Commit message: Expand camera list (add 'top' camera)

File: src/tunnel_inspection_sim/urdf/tunnel_robot.xacro (robot description, xacro)
@@ -58,5 +58,5 @@
   </joint>
   <joint name="left_camera_joint" type="fixed">
-    <origin xyz="0.1 0.05 0.1" rpy="0 -0.8 0.785"/>
+    <origin xyz="0.1 0.05 0.1" rpy="0 -0.55 1.05"/>
     <parent link="base_link"/>
     <child link="left_camera_link"/>
@@ -78,6 +78,27 @@
   </joint>
   <link name="left_camera_optical_frame"/>
+  <joint name="top_camera_joint" type="fixed">
+    <origin xyz="0.1 0 0.12" rpy="0 -1.35 0"/>
+    <parent link="base_link"/>
+    <child link="top_camera_link"/>
+  </joint>
+  <link name="top_camera_link">
+    <visual>
+      <geometry><box size="0.01 0.01 0.01"/></geometry>
+      <material name="dark_gray"><color rgba="0.2 0.2 0.2 1.0"/></material>
+    </visual>
+    <inertial>
+      <mass value="0.001"/>
+      <inertia ixx="0.00001" ixy="0" ixz="0" iyy="0.00001" iyz="0" izz="0.00001"/>
+    </inertial>
+  </link>
+  <joint name="top_camera_optical_joint" type="fixed">
+    <origin xyz="0 0 0" rpy="-1.5708 0 -1.5708"/>
+    <parent link="top_camera_link"/>
+    <child link="top_camera_optical_frame"/>
+  </joint>
+  <link name="top_camera_optical_frame"/>
   <joint name="right_camera_joint" type="fixed">
-    <origin xyz="0.1 -0.05 0.1" rpy="0 -0.8 -0.785"/>
+    <origin xyz="0.1 -0.05 0.1" rpy="0 -0.55 -1.05"/>
     <parent link="base_link"/>
     <child link="right_camera_link"/>
@@ -159,4 +180,24 @@
     </sensor>
   </gazebo>
+  <gazebo reference="top_camera_link">
+    <sensor name="top_rgbd_camera" type="rgbd_camera">
+      <topic>/top_camera</topic>
+      <gz_frame_id>top_camera_optical_frame</gz_frame_id>
+      <update_rate>15.0</update_rate>
+      <camera>
+        <horizontal_fov>1.57</horizontal_fov>
+        <image>
+          <width>640</width>
+          <height>480</height>
+        </image>
+        <clip>
+          <near>0.1</near>
+          <far>10.0</far>
+        </clip>
+      </camera>
+      <always_on>true</always_on>
+      <visualize>true</visualize>
+    </sensor>
+  </gazebo>
   <gazebo reference="right_camera_link">
     <sensor name="right_rgbd_camera" type="rgbd_camera">

Commit message: Make up for crack detection

File: src/tunnel_inspection_sim/urdf/tunnel_robot.xacro (robot description, xacro)
@@ -79,5 +79,5 @@
   <link name="left_camera_optical_frame"/>
   <joint name="top_camera_joint" type="fixed">
-    <origin xyz="0.1 0 0.12" rpy="0 -1.35 0"/>
+    <origin xyz="0.1 0 0.12" rpy="0 -1.45 0"/>
     <parent link="base_link"/>
     <child link="top_camera_link"/>

Commit message: Add a rear caster to the robot and adjust camera angle

File: src/tunnel_inspection_sim/urdf/tunnel_robot.xacro (robot description, xacro)
@@ -51,4 +51,13 @@
     <origin xyz="0.1 0 -0.07" rpy="0 0 0"/>
   </joint>
+  <link name="rear_caster_link">
+    <collision><geometry><sphere radius="0.03"/></geometry></collision>
+    <inertial><mass value="0.1"/><inertia ixx="0.0001" ixy="0" ixz="0" iyy="0.0001" iyz="0" izz="0.0001"/></inertial>
+  </link>
+  <joint name="rear_caster_joint" type="fixed">
+    <parent link="base_link"/>
+    <child link="rear_caster_link"/>
+    <origin xyz="-0.1 0 -0.07" rpy="0 0 0"/>
+  </joint>
   <link name="lidar_link"/>
   <joint name="lidar_joint" type="fixed">
@@ -58,5 +67,5 @@
   </joint>
   <joint name="left_camera_joint" type="fixed">
-    <origin xyz="0.1 0.05 0.1" rpy="0 -0.2882 1.05"/>
+    <origin xyz="0.1 0.05 0.1" rpy="0 -0.7854 0.7854"/>
     <parent link="base_link"/>
     <child link="left_camera_link"/>
@@ -79,5 +88,5 @@
   <link name="left_camera_optical_frame"/>
   <joint name="top_camera_joint" type="fixed">
-    <origin xyz="0.1 0 0.12" rpy="0 -1.1882 0"/>
+    <origin xyz="0.1 0 0.12" rpy="0 -1.5708 0"/>
     <parent link="base_link"/>
     <child link="top_camera_link"/>
@@ -100,5 +109,5 @@
   <link name="top_camera_optical_frame"/>
   <joint name="right_camera_joint" type="fixed">
-    <origin xyz="0.1 -0.05 0.1" rpy="0 -0.2882 -1.05"/>
+    <origin xyz="0.1 -0.05 0.1" rpy="0 -0.7854 -0.7854"/>
     <parent link="base_link"/>
     <child link="right_camera_link"/>
@@ -135,4 +144,8 @@
   </gazebo>
   <gazebo reference="caster_link">
+    <mu1>0.0</mu1>
+    <mu2>0.0</mu2>
+  </gazebo>
+  <gazebo reference="rear_caster_link">
     <mu1>0.0</mu1>
     <mu2>0.0</mu2>

Commit message: Update: increase tunnel size & tune camera pos.

File: src/tunnel_inspection_sim/urdf/tunnel_robot.xacro (robot description, xacro)
@@ -67,5 +67,5 @@
   </joint>
   <joint name="left_camera_joint" type="fixed">
-    <origin xyz="0.1 0.05 0.1" rpy="0 -0.7854 0.7854"/>
+    <origin xyz="0.18 0.17 0.11" rpy="0 -0.28 1.25"/>
     <parent link="base_link"/>
     <child link="left_camera_link"/>
@@ -88,5 +88,5 @@
   <link name="left_camera_optical_frame"/>
   <joint name="top_camera_joint" type="fixed">
-    <origin xyz="0.1 0 0.12" rpy="0 -1.5708 0"/>
+    <origin xyz="0.16 0 0.10" rpy="0 -1.5708 0"/>
     <parent link="base_link"/>
     <child link="top_camera_link"/>
@@ -109,5 +109,5 @@
   <link name="top_camera_optical_frame"/>
   <joint name="right_camera_joint" type="fixed">
-    <origin xyz="0.1 -0.05 0.1" rpy="0 -0.7854 -0.7854"/>
+    <origin xyz="0.18 -0.17 0.11" rpy="0 -0.28 -1.25"/>
     <parent link="base_link"/>
     <child link="right_camera_link"/>
@@ -179,5 +179,5 @@
       <update_rate>15.0</update_rate>
       <camera>
-        <horizontal_fov>1.57</horizontal_fov>
+        <horizontal_fov>1.70</horizontal_fov>
         <image>
           <width>640</width>
@@ -185,6 +185,6 @@
         </image>
         <clip>
-          <near>0.1</near>
-          <far>10.0</far>
+          <near>0.05</near>
+          <far>1.3</far>
         </clip>
       </camera>
@@ -199,5 +199,5 @@
       <update_rate>15.0</update_rate>
       <camera>
-        <horizontal_fov>1.57</horizontal_fov>
+        <horizontal_fov>1.92</horizontal_fov>
         <image>
           <width>640</width>
@@ -205,6 +205,6 @@
         </image>
         <clip>
-          <near>0.1</near>
-          <far>10.0</far>
+          <near>0.05</near>
+          <far>1.3</far>
         </clip>
       </camera>
@@ -219,5 +219,5 @@
       <update_rate>15.0</update_rate>
       <camera>
-        <horizontal_fov>1.57</horizontal_fov>
+        <horizontal_fov>1.70</horizontal_fov>
         <image>
           <width>640</width>
@@ -225,6 +225,6 @@
         </image>
         <clip>
-          <near>0.1</near>
-          <far>10.0</far>
+          <near>0.05</near>
+          <far>1.3</far>
         </clip>
       </camera>
